File: cam-to-rs485-avr/board/jvc.sch (KiCad schematic (older format))
At the start: 31 parts, among them J1 Conn_01x03, J2 Conn_02x03_Odd_Even, J3 Conn_01x04, J4 Conn_01x02, Q1 BC847, U1 MAX485E, U2 L78L05_SOT89, U3 ATtiny2313-20SU, Y1 Crystal

Commit message: 485 Verlängerung as subprojekt fertig
code könnte schöner werden, sehr viel hartkodiert
Parts:
- U1: footprint (none) -> Package_DIP:DIP-8_W7.62mm_Socket
- U3: symbol jvc-rescue:ATtiny2313-20SU-MCU_Microchip_ATtiny -> jvc-rescue:ATtiny2313-20SU-MCU_Microchip_ATtiny-jvc-rescue
Changed lines of the file:
@@
 $EndDescr
 $Comp
-L jvc-rescue:ATtiny2313-20SU-MCU_Microchip_ATtiny U3
+L jvc-rescue:ATtiny2313-20SU-MCU_Microchip_ATtiny-jvc-rescue U3
 U 1 1 5C6F4FFC
 P 5550 3850
@@
 F 0 "U1" H 3400 5628 50  0000 C CNN
 F 1 "MAX485E" H 3400 5537 50  0000 C CNN
-F 2 "" H 3400 4250 50  0001 C CNN
+F 2 "Package_DIP:DIP-8_W7.62mm_Socket" H 3400 4250 50  0001 C CNN
 F 3 "https://datasheets.maximintegrated.com/en/ds/MAX1487E-MAX491E.pdf" H 3400 5000 50  0001 C CNN
 	1    3400 4950
@@
 Connection ~ 2800 4850
 Wire Wire Line
-	3400 5600 3400 5550
+	3400 5550 3400 5600
 $EndSCHEMATC
